File: PCB/FullPCB/EEGFrontOnly.brd (EAGLE design)
At the start: 87.5 x 46.7 mm, 118 parts, among them IC1 ADS1299-X, U1 LP2985-33DBVT, U10 HT7318, U11 TMS320F28335PGFA, U12 HT7333, U13 2.93V, U14 MAX811-812, U2 B0505S-1WB0505S-1W, U3 TPS60403DBVT, U4 TPS73225DBVR, U5 TPS73225DBVR, U6 TPD4E1B06DCKR, U7 TPD4E1B06DCKR, U8 TPD4E1B06DCKR, U9 HT7333

Commit message: update main pcb
Parts:
- added J8: JTAG, SparkFun-Connectors:2X7
- added R25, R26, R27, R28, R29, R30: 10k, SparkFun-Resistors:0402
- moved C58 66.7 mm to (-2.29, 14.7), turned to 270 degrees
- moved C57 58.0 mm to (-2.29, 6.99), turned to 90 degrees
- moved Y1 56.9 mm to (-3.17, 10.8), turned to 90 degrees
- moved C53 7.55 mm to (6.99, -10.7)
- moved U10 7.27 mm to (11.0, -9.14)
- moved C54 7.20 mm to (15.1, -10.7)
- moved C52 0.40 mm to (-3.68, -11.0)
- moved C51 0.13 mm to (-12.1, -11.0)
Connections:
- removed net VDD: U11.61
- removed net VDDIO: U11.71
- removed net VDDIO_2: U11.9
- removed net VDD_2: U11.15
- removed net VDD_3: U11.4
- removed net VDD_4: U11.23
- removed net VDD_5: U11.29
- net GND: now also U11.103, U11.105, U11.106, U11.108, U11.118, U11.120, U11.125, U11.14, U11.140, U11.144, U11.147, U11.155, U11.160, U11.166, U11.171, U11.22, U11.3, U11.30, U11.60, U11.70, U11.8, U11.83, U11.92
- net VCC_1V8: now also U11.15, U11.23, U11.29, U11.4, U11.61
- net VCC_DSP: now also U11.71, U11.9
