File: PCB/FullPCB/EEGFrontOnly.sch (EAGLE design)
At the start: 114 parts, among them IC1 ADS1299-X, U1 LP2985-33DBVT, U10 HT7318, U11 TMS320F28335PGFA, U12 HT7333, U13 2.93V, U14 MAX811-812, U2 B0505S-1WB0505S-1W, U3 TPS60403DBVT, U4 TPS73225DBVR, U5 TPS73225DBVR, U6 TPD4E1B06DCKR, U7 TPD4E1B06DCKR, U8 TPD4E1B06DCKR, U9 HT7333

Commit message: update main pcb
Parts:
- added J8: JTAG, SparkFun-Connectors:CONN_07X2
- added R25, R26, R27, R28, R29, R30: 10k, SparkFun-Resistors:10KOHM-0402-1/10W-1%
Connections:
- net GND: now also U11A.VSS, U11A.VSS_2, U11A.VSS_3, U11A.VSS_4, U11A.VSS_5, U11A.VSS_6, U11A.VSS_7, U11A.VSS_8, U11B.VSS, U11B.VSS_10, U11B.VSS_11, U11B.VSS_12, U11B.VSS_13, U11B.VSS_14, U11B.VSS_2, U11B.VSS_3, U11B.VSS_4, U11B.VSS_5, U11B.VSS_6, U11B.VSS_7, U11B.VSS_8, U11B.VSS_9, U11B.XCLKIN
- net VCC_1V8: now also U11A.VDD, U11A.VDD_2, U11A.VDD_3, U11A.VDD_4, U11A.VDD_5
- net VCC_DSP: now also U11A.VDDIO, U11A.VDDIO_2
Changed lines of the file:
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@@
 <part name="C58" library="SparkFun-Capacitors" deviceset="22PF" device="-0402-50V-5%" value="22pF"/>
 <part name="GND16" library="SparkFun-PowerSymbols" deviceset="GND2" device=""/>
+<part name="GND17" library="SparkFun-PowerSymbols" deviceset="GND2" device=""/>
+<part name="GND18" library="SparkFun-PowerSymbols" deviceset="GND2" device=""/>
+<part name="J8" library="SparkFun-Connectors" deviceset="CONN_07X2" device="" value="JTAG"/>
+<part name="R25" library="SparkFun-Resistors" deviceset="10KOHM" device="-0402-1/10W-1%" value="10k"/>
+<part name="R26" library="SparkFun-Resistors" deviceset="10KOHM" device="-0402-1/10W-1%" value="10k"/>
+<part name="R27" library="SparkFun-Resistors" deviceset="10KOHM" device="-0402-1/10W-1%" value="10k"/>
+<part name="R28" library="SparkFun-Resistors" deviceset="10KOHM" device="-0402-1/10W-1%" value="10k"/>
+<part name="R29" library="SparkFun-Resistors" deviceset="10KOHM" device="-0402-1/10W-1%" value="10k"/>
+<part name="R30" library="SparkFun-Resistors" deviceset="10KOHM" device="-0402-1/10W-1%" value="10k"/>
 </parts>
 <sheets>
@@
 <instance part="C58" gate="G$1" x="185.42" y="119.38" rot="R90"/>
 <instance part="GND16" gate="G$1" x="172.72" y="102.87"/>
+<instance part="GND17" gate="G$1" x="-5.08" y="3.81"/>
+<instance part="GND18" gate="G$1" x="193.04" y="67.31"/>
+<instance part="J8" gate="G$1" x="337.82" y="101.6"/>
+<instance part="R25" gate="G$1" x="320.04" y="116.84" rot="R90"/>
+<instance part="R26" gate="G$1" x="312.42" y="116.84" rot="R90"/>
+<instance part="R27" gate="G$1" x="304.8" y="116.84" rot="R90"/>
+<instance part="R28" gate="G$1" x="297.18" y="116.84" rot="R90"/>
+<instance part="R29" gate="G$1" x="355.6" y="109.22" rot="R90"/>
+<instance part="R30" gate="G$1" x="368.3" y="116.84" rot="R90"/>
 </instances>
 <busses>
@@
 <pinref part="C58" gate="G$1" pin="1"/>
 <wire x1="180.34" y1="119.38" x2="172.72" y2="119.38" width="0.1524" layer="91"/>
-<wire x1="172.72" y1="119.38" x2="172.72" y2="109.22" width="0.1524" layer="91"/>
+<wire x1="172.72" y1="119.38" x2="172.72" y2="111.76" width="0.1524" layer="91"/>
 <pinref part="C57" gate="G$1" pin="1"/>
+<wire x1="172.72" y1="111.76" x2="172.72" y2="109.22" width="0.1524" layer="91"/>
 <wire x1="172.72" y1="109.22" x2="180.34" y2="109.22" width="0.1524" layer="91"/>
 <pinref part="GND16" gate="G$1" pin="3.3V"/>
 <wire x1="172.72" y1="105.41" x2="172.72" y2="109.22" width="0.1524" layer="91"/>
 <junction x="172.72" y="109.22"/>
+<pinref part="U11" gate="B" pin="XCLKIN"/>
+<wire x1="198.12" y1="111.76" x2="172.72" y2="111.76" width="0.1524" layer="91"/>
+<junction x="172.72" y="111.76"/>
+</segment>
+<segment>
+<pinref part="GND17" gate="G$1" pin="3.3V"/>
+<pinref part="U11" gate="A" pin="VSS"/>
+<wire x1="-5.08" y1="6.35" x2="-5.08" y2="7.62" width="0.1524" layer="91"/>
+<wire x1="-5.08" y1="7.62" x2="0" y2="7.62" width="0.1524" layer="91"/>
+<pinref part="U11" gate="A" pin="VSS_2"/>
+<wire x1="0" y1="7.62" x2="2.54" y2="7.62" width="0.1524" layer="91"/>
+<wire x1="2.54" y1="25.4" x2="0" y2="25.4" width="0.1524" layer="91"/>
+<wire x1="0" y1="25.4" x2="0" y2="22.86" width="0.1524" layer="91"/>
+<junction x="0" y="7.62"/>
+<pinref part="U11" gate="A" pin="VSS_3"/>
+<wire x1="0" y1="22.86" x2="0" y2="20.32" width="0.1524" layer="91"/>
+<wire x1="0" y1="20.32" x2="0" y2="17.78" width="0.1524" layer="91"/>
+<wire x1="0" y1="17.78" x2="0" y2="15.24" width="0.1524" layer="91"/>
+<wire x1="0" y1="15.24" x2="0" y2="12.7" width="0.1524" layer="91"/>
+<wire x1="0" y1="12.7" x2="0" y2="10.16" width="0.1524" layer="91"/>
+<wire x1="0" y1="10.16" x2="0" y2="7.62" width="0.1524" layer="91"/>
+<wire x1="2.54" y1="22.86" x2="0" y2="22.86" width="0.1524" layer="91"/>
+<junction x="0" y="22.86"/>
+<pinref part="U11" gate="A" pin="VSS_4"/>
+<wire x1="2.54" y1="20.32" x2="0" y2="20.32" width="0.1524" layer="91"/>
+<junction x="0" y="20.32"/>
+<pinref part="U11" gate="A" pin="VSS_5"/>
+<wire x1="2.54" y1="17.78" x2="0" y2="17.78" width="0.1524" layer="91"/>
+<junction x="0" y="17.78"/>
+<pinref part="U11" gate="A" pin="VSS_6"/>
+<wire x1="2.54" y1="15.24" x2="0" y2="15.24" width="0.1524" layer="91"/>
+<junction x="0" y="15.24"/>
+<pinref part="U11" gate="A" pin="VSS_7"/>
+<wire x1="2.54" y1="12.7" x2="0" y2="12.7" width="0.1524" layer="91"/>
+<junction x="0" y="12.7"/>
+<pinref part="U11" gate="A" pin="VSS_8"/>
+<wire x1="2.54" y1="10.16" x2="0" y2="10.16" width="0.1524" layer="91"/>
+<junction x="0" y="10.16"/>
+</segment>
+<segment>
+<pinref part="U11" gate="B" pin="VSS_2"/>
+<wire x1="198.12" y1="106.68" x2="193.04" y2="106.68" width="0.1524" layer="91"/>
+<pinref part="GND18" gate="G$1" pin="3.3V"/>
+<wire x1="193.04" y1="106.68" x2="193.04" y2="104.14" width="0.1524" layer="91"/>
+<pinref part="U11" gate="B" pin="VSS_3"/>
+<wire x1="193.04" y1="104.14" x2="193.04" y2="101.6" width="0.1524" layer="91"/>
+<wire x1="193.04" y1="101.6" x2="193.04" y2="99.06" width="0.1524" layer="91"/>
+<wire x1="193.04" y1="99.06" x2="193.04" y2="96.52" width="0.1524" layer="91"/>
+<wire x1="193.04" y1="96.52" x2="193.04" y2="93.98" width="0.1524" layer="91"/>
+<wire x1="193.04" y1="93.98" x2="193.04" y2="91.44" width="0.1524" layer="91"/>
+<wire x1="193.04" y1="91.44" x2="193.04" y2="88.9" width="0.1524" layer="91"/>
+<wire x1="193.04" y1="88.9" x2="193.04" y2="86.36" width="0.1524" layer="91"/>
+<wire x1="193.04" y1="86.36" x2="193.04" y2="83.82" width="0.1524" layer="91"/>
+<wire x1="193.04" y1="83.82" x2="193.04" y2="81.28" width="0.1524" layer="91"/>
+<wire x1="193.04" y1="81.28" x2="193.04" y2="78.74" width="0.1524" layer="91"/>
+<wire x1="193.04" y1="78.74" x2="193.04" y2="76.2" width="0.1524" layer="91"/>
+<wire x1="193.04" y1="76.2" x2="193.04" y2="73.66" width="0.1524" layer="91"/>
+<wire x1="193.04" y1="73.66" x2="193.04" y2="69.85" width="0.1524" layer="91"/>
+<wire x1="198.12" y1="104.14" x2="193.04" y2="104.14" width="0.1524" layer="91"/>
+<junction x="193.04" y="104.14"/>
+<pinref part="U11" gate="B" pin="VSS_4"/>
+<wire x1="198.12" y1="101.6" x2="193.04" y2="101.6" width="0.1524" layer="91"/>
+<junction x="193.04" y="101.6"/>
+<pinref part="U11" gate="B" pin="VSS_5"/>
+<wire x1="198.12" y1="99.06" x2="193.04" y2="99.06" width="0.1524" layer="91"/>
+<junction x="193.04" y="99.06"/>
+<pinref part="U11" gate="B" pin="VSS_6"/>
+<wire x1="198.12" y1="96.52" x2="193.04" y2="96.52" width="0.1524" layer="91"/>
+<junction x="193.04" y="96.52"/>
+<pinref part="U11" gate="B" pin="VSS_7"/>
+<wire x1="198.12" y1="93.98" x2="193.04" y2="93.98" width="0.1524" layer="91"/>
+<junction x="193.04" y="93.98"/>
+<pinref part="U11" gate="B" pin="VSS_8"/>
+<wire x1="198.12" y1="91.44" x2="193.04" y2="91.44" width="0.1524" layer="91"/>
+<junction x="193.04" y="91.44"/>
+<pinref part="U11" gate="B" pin="VSS_9"/>
+<wire x1="198.12" y1="88.9" x2="193.04" y2="88.9" width="0.1524" layer="91"/>
+<junction x="193.04" y="88.9"/>
+<pinref part="U11" gate="B" pin="VSS_10"/>
+<wire x1="198.12" y1="86.36" x2="193.04" y2="86.36" width="0.1524" layer="91"/>
+<junction x="193.04" y="86.36"/>
+<pinref part="U11" gate="B" pin="VSS_11"/>
+<wire x1="198.12" y1="83.82" x2="193.04" y2="83.82" width="0.1524" layer="91"/>
+<junction x="193.04" y="83.82"/>
+<pinref part="U11" gate="B" pin="VSS_12"/>
+<wire x1="198.12" y1="81.28" x2="193.04" y2="81.28" width="0.1524" layer="91"/>
+<junction x="193.04" y="81.28"/>
+<pinref part="U11" gate="B" pin="VSS_13"/>
+<wire x1="198.12" y1="78.74" x2="193.04" y2="78.74" width="0.1524" layer="91"/>
+<junction x="193.04" y="78.74"/>
+<pinref part="U11" gate="B" pin="VSS_14"/>
+<wire x1="198.12" y1="76.2" x2="193.04" y2="76.2" width="0.1524" layer="91"/>
+<junction x="193.04" y="76.2"/>
+<pinref part="U11" gate="B" pin="VSS"/>
+<wire x1="198.12" y1="73.66" x2="193.04" y2="73.66" width="0.1524" layer="91"/>
+<junction x="193.04" y="73.66"/>
 </segment>
 </net>
@@
 <junction x="190.5" y="142.24"/>
 </segment>
+<segment>
+<pinref part="U11" gate="A" pin="VDD_2"/>
+<wire x1="2.54" y1="157.48" x2="0" y2="157.48" width="0.1524" layer="91"/>
+<wire x1="0" y1="157.48" x2="-2.54" y2="157.48" width="0.1524" layer="91"/>
+<wire x1="-2.54" y1="157.48" x2="-2.54" y2="160.02" width="0.1524" layer="91"/>
+<wire x1="-2.54" y1="160.02" x2="-7.62" y2="160.02" width="0.1524" layer="91"/>
+<label x="-7.62" y="160.02" size="1.778" layer="95" rot="R180" xref="yes"/>
+<pinref part="U11" gate="A" pin="VDD"/>
+<wire x1="2.54" y1="147.32" x2="0" y2="147.32" width="0.1524" layer="91"/>
+<wire x1="0" y1="147.32" x2="0" y2="149.86" width="0.1524" layer="91"/>
+<junction x="0" y="157.48"/>
+<pinref part="U11" gate="A" pin="VDD_3"/>
+<wire x1="0" y1="149.86" x2="0" y2="152.4" width="0.1524" layer="91"/>
+<wire x1="0" y1="152.4" x2="0" y2="154.94" width="0.1524" layer="91"/>
+<wire x1="0" y1="154.94" x2="0" y2="157.48" width="0.1524" layer="91"/>
+<wire x1="2.54" y1="154.94" x2="0" y2="154.94" width="0.1524" layer="91"/>
+<junction x="0" y="154.94"/>
+<pinref part="U11" gate="A" pin="VDD_4"/>
+<wire x1="2.54" y1="152.4" x2="0" y2="152.4" width="0.1524" layer="91"/>
+<junction x="0" y="152.4"/>
+<pinref part="U11" gate="A" pin="VDD_5"/>
+<wire x1="2.54" y1="149.86" x2="0" y2="149.86" width="0.1524" layer="91"/>
+<junction x="0" y="149.86"/>
+</segment>
 </net>
 <net name="VCC_DSP" class="0">
@@
 <junction x="190.5" y="124.46"/>
 </segment>
-</net>
+<segment>
+<pinref part="U11" gate="A" pin="VDDIO_2"/>
+<wire x1="2.54" y1="144.78" x2="-2.54" y2="144.78" width="0.1524" layer="91"/>
+<wire x1="-2.54" y1="144.78" x2="-2.54" y2="149.86" width="0.1524" layer="91"/>
+<wire x1="-2.54" y1="149.86" x2="-7.62" y2="149.86" width="0.1524" layer="91"/>
+<label x="-7.62" y="149.86" size="1.778" layer="95" rot="R180" xref="yes"/>
+<pinref part="U11" gate="A" pin="VDDIO"/>
+<wire x1="2.54" y1="139.7" x2="-2.54" y2="139.7" width="0.1524" layer="91"/>
+<wire x1="-2.54" y1="139.7" x2="-2.54" y2="144.78" width="0.1524" layer="91"/>
+<junction x="-2.54" y="144.78"/>
+</segment>
+</net>

Commit message: update pcb & update dsp main code
Parts:
- added C59, C60, C61, C62, C63, C64, C65, C66, C67, C68, C69, C70, C71, C72, C73, C74, C75, C76, C77: 0.1uF, SparkFun-Capacitors:0.1UF-0402-16V-10%
- added C78, C79: 22pF, SparkFun-Capacitors:22PF-0402-50V-5%
- added J11: MICRO-SD_CARD_SOCKET, SparkFun-Connectors:MICRO-SD_CARD_SOCKET
- added R31, R32, R33: 0OHM, SparkFun-Resistors:0OHM
- added U$3: CH340G, ch340g:CH340G
- added Y2: 12MHz, SparkFun-Clocks:CRYSTALSMD-3.2X2.5
- C39, C48: value 4.7nF -> 0.1uF; device SparkFun-Capacitors:4.7NF-0402 -> SparkFun-Capacitors:0.1UF-0402-16V-10%
- J2: value (none) -> USB_B_PTH; device SparkFun-Connectors:USB_MICRO-BREDUCED_PASTE -> SparkFun-Connectors:USB_B_PTH
- R4: value 4.99K -> 0OHM; device SparkFun-Resistors:4.99KOHM-0402 -> SparkFun-Resistors:0OHM
- Y1: value (none) -> 30MHz
Connections:
- removed net VCC_1V8: C54.1, U10.OUT, U11A.VDD, U11A.VDD_2, U11A.VDD_3, U11A.VDD_4, U11A.VDD_5, U11B.VDD, U11B.VDD_2, U11B.VDD_3, U11B.VDD_4, U11B.VDD_5, U11B.VDD_6, U11B.VDD_7, U11B.VDD_8
- removed net VCC_DSP: C52.1, C53.1, C55.1, R23.2, R24.2, U10.IN, U11A.VDDIO, U11A.VDDIO_2, U11B.VDDIO, U11B.VDDIO_2, U11B.VDDIO_3, U11B.VDDIO_4, U11B.VDDIO_5, U11B.VDDIO_6, U12.OUT, U13.VCC, U14.VCC
- new net 1.8V: C39.1, C48.1, C54.1, C59.1, C60.1, C61.1, C62.1, C63.1, C64.1, C65.1, C74.1, C75.1, C76.1, C77.1, R4.1, U10.OUT, U11A.VDD, U11A.VDD_2, U11A.VDD_3, U11A.VDD_4, U11A.VDD_5, U11B.VDD, U11B.VDD_2, U11B.VDD_3, U11B.VDD_4, U11B.VDD_5, U11B.VDD_6, U11B.VDD_7, U11B.VDD_8
- new net 3.3V: C52.1, C53.1, C55.1, C66.1, C67.1, C68.1, C69.1, C70.1, C71.1, C72.1, C73.1, J8.5, R23.2, R24.2, R25.2, R26.2, R27.2, R28.2, R30.2, R31.1, R32.1, U$3.V3, U10.IN, U11A.VDDIO, U11A.VDDIO_2, U11B.VDDIO, U11B.VDDIO_2, U11B.VDDIO_3, U11B.VDDIO_4, U11B.VDDIO_5, U11B.VDDIO_6, U12.OUT, U13.VCC, U14.VCC
- new net A1V8: R4.2, U11A.VDD1A18, U11A.VDD2A18
- new net A3V3: R31.2, U11A.VDDA2, U11A.VDDAIO
- new net D+_ISO: U$3.D+
- new net D-_ISO: U$3.D-
- new net EMU0: J8.13, R28.1, U11A.EMU0
- new net EMU1: J8.14, R30.1, U11A.EMU1
- new net GNDA: R33.2, U11A.VSS1AGND, U11A.VSS2AGND, U11A.VSSA2, U11A.VSSAIO
- new net N$32: C40.2, C41.2, C42.2, C43.2, C44.2, C45.2, C46.2, C47.2, IC1.SRB1, J5.2, R13.2
- new net N$33: U$3.TX
- new net N$34: U$3.RX
- new net TCK: J8.11, J8.9, R27.1, U11A.TCK
- new net TDI: J8.3, R26.1, U11A.TDI
- new net TDO: J8.7, U11A.TDO
- new net TMS: J8.1, R25.1, U11A.TMS
- new net TRST: J8.2, R29.2, U11A.~TRST
- new net VDD3VFL: R32.2, U11A.VDD3VFL
- net AGND: no longer C39.2, C40.2, C41.2, C42.2, C43.2, C44.2, C45.2, C46.2, C47.2, C48.2
- net GND: now also C39.2, C48.2, C59.2, C60.2, C61.2, C62.2, C63.2, C64.2, C65.2, C66.2, C67.2, C68.2, C69.2, C70.2, C71.2, C72.2, C73.2, C74.2, C75.2, C76.2, C77.2, C78.1, C79.1, J8.10, J8.12, J8.4, J8.8, R29.1, R33.1, U$3.GND
- net N$12: now also C78.2, U$3.XI, Y2.2; no longer C48.1, IC1.SRB1, J5.2, R13.2
- net N$14: now also C79.2, U$3.XO, Y2.1; no longer C38.1, C39.1, IC1.BIASIN, IC1.BIASOUT, R3.2, R4.2
- net P_BIAS: now also C38.1, IC1.BIASIN, IC1.BIASOUT, R3.2; no longer R4.1
- net RST_DSP: now also U11A.~XRS
- net SPI_CLK: now also U11B.GPIO56/SPICLKA/XD23
- net SPI_CS: now also U11B.GPIO57/~SPISTEA/XD22
- net SPI_MISO: now also U11B.GPIO55/SPISOMIA/XD24
- net SPI_MOSI: now also U11B.GPIO54/SPISIMOA/XD25
Other:
- moved on the sheet: R29, R30

Commit message: update main pcb
Parts:
- added C80, C81, C82, C83, C84, C85, C86, C87, C88, C89: 0.1uF, SparkFun-Capacitors:0.1UF-0402-16V-10%
- added D2, D3: RED, SparkFun-LED:LED-RED0603
- added IC2: ADUM4160BRWZ, SOIC127P1032X265-16N:ADUM4160BRWZ
- added J12, J13, J14, J15: 455-1750-1-ND, SparkFun-Connectors:CONN_03
- added R34, R35, R41, R42, R43, R44: 4.7k, SparkFun-Resistors:4.7KOHM-0402-1/10W-1%
- added R36, R37, R38, R39, R40, R49, R50, R51, R52: 22, SparkFun-Resistors:22OHM-0402-1/10W-1%
- added R45, R46, R47, R48: 1k, SparkFun-Resistors:1KOHM-0402-1%
- added R53, R54, R55, R56: 10k, SparkFun-Resistors:10KOHM-0402-1/10W-1%
- added S3: (no value), switch-dil:DIP04S
- R17, R18, R19, R20: value 22 -> 0OHM; device SparkFun-Resistors:22OHM-0402-1/10W-1% -> SparkFun-Resistors:0OHM
Connections:
- removed net D+_ISO: U$3.D+
- removed net D-_ISO: U$3.D-
- new net D_ISO_N: R51.2, U$3.D-
- new net D_ISO_P: R52.2, U$3.D+
- new net D_ISO_PRE_N: IC2.DD-, R51.1
- new net D_ISO_PRE_P: IC2.DD+, R52.1
- new net D_N: J2.D-, R49.1
- new net D_P: J2.D+, R50.1
- new net N$35: R36.1, U11B.GPIO54/SPISIMOA/XD25
- new net N$36: IC2.UD-, R49.2
- new net N$37: R37.1, U11B.GPIO55/SPISOMIA/XD24
- new net N$38: R38.1, U11B.GPIO56/SPICLKA/XD23
- new net N$39: R39.1, U11B.GPIO57/~SPISTEA/XD22
- new net N$40: R40.1, U11A.GPIO16/SPISIMOA/CANTXB/~TZ5
- new net N$41: IC2.UD+, R50.2
- new net N$54: R48.1, S3-4.2
- new net N$55: R47.1, S3-3.2
- new net N$56: R46.1, S3-2.2
- new net N$57: R45.1, S3-1.2
- new net PIN: IC2.PIN
- new net RX: D2.C, J13.1, U$3.TX, U11A.GPIO11/EPWM6B/SCIRXDB/ECAP4
- new net SPD: IC2.SPD, J15.2
- new net SPI_CS_MIRCOSD: J11.!CS, R40.2, R56.1
- new net SPU: IC2.SPU, J14.2
- new net TX: D3.C, J13.2, U$3.RX, U11A.GPIO9/EPWM5B/SCITXDB/ECAP3
- new net VCC_CH340: C80.1, J12.2, R34.2, R35.2, U$3.VCC
- new net XA12: R41.2, S3-1.1, U11B.GPIO84/XA12
- new net XA13: R42.2, S3-2.1, U11B.GPIO85/XA13
- new net XA14: R43.2, S3-3.1, U11B.GPIO86/XA14
- new net XA15: R44.2, S3-4.1, U11B.GPIO87/XA15
- net 3.3V: now also C83.1, C84.1, IC2.VBUS2, IC2.VDD2, J11.VCC, J12.3, J15.3, R41.1, R42.1, R43.1, R44.1, R53.2, R54.2, R55.2, R56.2
- net A1V8: now also C85.1, C86.1
- net A3V3: now also C87.1, C88.1
- net GND: now also C80.2, C83.2, C84.2, C89.2, IC2.GND2, J11.GND, J11.SHIELD@1, J11.SHIELD@3, J13.3, J15.1, R45.2, R46.2, R47.2, R48.2
- net GND-ISO: now also C81.2, C82.2, IC2.GND1, J14.1
- net GNDA: now also C85.2, C86.2, C87.2, C88.2
- net N$33: now also D2.A, R34.1; no longer U$3.TX
- net N$34: now also D3.A, R35.1; no longer U$3.RX
- net PWD: now also U11B.GPIO63/SCITXDC/XD16
- net RST: now also U11B.GPIO62/SCIRXDC/XD17
- net SPI_CLK: now also J11.SCK, R38.2, R55.1; no longer U11B.GPIO56/SPICLKA/XD23
- net SPI_CS: now also R39.2; no longer U11B.GPIO57/~SPISTEA/XD22
- net SPI_DRDY: now also U11A.GPIO15/~TZ4/~XHOLDA/SCIRXDB/MFSXB
- net SPI_MISO: now also J11.DO, R37.2, R54.1; no longer U11B.GPIO55/SPISOMIA/XD24
- net SPI_MOSI: now also J11.DI, R36.2, R53.1; no longer U11B.GPIO54/SPISIMOA/XD25
- net SPI_START: now also U11A.GPIO17/SPISOMIA/CANRXB/~TZ6
- net VBAT: now also J12.1
- net VCC-ISO: now also C81.1, IC2.VBUS1
- net VCCIO: now also C82.1, IC2.PDEN, IC2.VDD1, J14.3
- net VDD3VFL: now also C89.1
Other:
- moved on the sheet: C39, C48, C59, C60, C61, C62, C63, C64, C65, C74, C75, C76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

Commit message: full pcb nearly complete
Parts:
- added C90, C91: 2.2uF, SparkFun-Capacitors:2.2UF-0402-10V-20%
- added D10, D11, D4, D5, D6, D7, D8, D9: RED, SparkFun-LED:LED-RED0603
- added R57, R58, R59, R60, R61, R62, R63, R64: 1k, SparkFun-Resistors:1KOHM-0402-1%
- added R65: 22k, SparkFun-Resistors:22KOHM0402-1/10W-1%
Connections:
- net N$32 renamed EEG_REF
- new net LED1: D4.C, U11A.GPIO0/EPWM1A
- new net LED2: D5.C, U11A.GPIO1/EPWM1B/ECAP6/MFSRB
- new net LED3: D6.C, U11A.GPIO2/EPWM2A
- new net LED4: D7.C, U11A.GPIO5/EPWM3B/MFSRA/ECAP1
- new net LED5: D8.C, U11A.GPIO4/EPWM3A
- new net LED6: D9.C, U11A.GPIO3/EPWM2B/ECAP5/MCLKRB
- new net LED7: D10.C, U11A.GPIO12/~TZ1/CANTXB/MDXB
- new net LED8: D11.C, U11B.GPIO36/SCIRXDA/~XZCS0
- new net N$32: D11.A, R64.1
- new net N$42: D10.A, R63.1
- new net N$43: D9.A, R62.1
- new net N$44: D8.A, R61.1
- new net N$45: D7.A, R60.1
- new net N$46: D6.A, R59.1
- new net N$47: D5.A, R58.1
- new net N$48: D4.A, R57.1
- new net N$49: C90.1, U11A.ADCREFP
- new net N$50: C91.1, U11A.ADCREFM
- new net N$51: R65.2, U11A.ADCRESEXT
- new net SDCARD_CD: J11.CD1, J11.CD2, U11B.GPIO51/EQEP1B/XD28
- net 3.3V: now also R57.2, R58.2, R59.2, R60.2, R61.2, R62.2, R63.2, R64.2
- net GNDA: now also C90.2, C91.2, R65.1, U11A.ADCLO, U11A.ADCREFIN
Other:
- moved on the sheet: J11

Commit message: full pcb nearly complete
Parts:
- added J16, J17: (no value), SparkFun-Connectors:CONN_02
Connections:
- net GND: now also J16.2
- net GND-ISO: now also J16.1
- net VBATPRE: now also J17.2
- net VCC-ISO: now also J17.1
Other:
- moved on the sheet: C55, C56, D1, R21, R22, R23, R24, S2, U13, U14
