File: PCB/FullPCB/EEGFull.brd (EAGLE design)
At the start: 87.4 x 92.6 mm, 215 parts, among them IC1 ADS1299-X, IC2 ADUM4160BRWZ, J11 MICRO-SD_CARD_SOCKET, J12 455-1750-1-ND, J13 455-1750-1-ND, J14 455-1750-1-ND, J15 455-1750-1-ND, J2 USB_B_PTH, J8 JTAG, U1 LP2985-33DBVT, U10 HT7318, U11 TMS320F28335PGFA, U12 HT7333, U13 2.93V, U14 MAX811-812, U2 B0505S-1WB0505S-1W, U3 TPS60403DBVT, U4 TPS73225DBVR, U5 TPS73225DBVR, U6 TPD4E1B06DCKR, U7 TPD4E1B06DCKR, U8 TPD4E1B06DCKR, U9 HT7333, Y1 30MHz, Y2 12MHz

Commit message: update Full PCB
Parts:
- added C92, C93, C94: 0.1uF, SparkFun-Capacitors:0402
- added C95, C96: 4.7uF, SparkFun-Capacitors:0603
- added F1: 6V/2A, SparkFun-Fuses:1206
- added J18: (no value), SparkFun-Connectors:1X02
- added J19: (no value), SparkFun-Connectors:SCREWTERMINAL-3.5MM-2
- added L5, L6: 3.3µH/±20%/450mA, SparkFun-Coils:0805
- added R66: 10k, SparkFun-Resistors:0402
- added U15: ISO721D, Texas Instruments_By_element14_Batch_1:SOIC127P600X175-8N
- U2: value B0505S-1WB0505S-1W -> (none); device jingjieparts:DIP4 -> jingjieparts:SIP
- moved U2 11.5 mm to (39.8, 89.1)
Connections:
- removed net PIN: IC2.12
- new net ISO_IN: J19.2, U15.2
- new net MR: C92.1, J18.1, R24.1, S2.3, U14.3
- new net N$52: C95.1, L5.2, U2.VIN
- new net N$58: L6.1, U2.VO
- new net TRIGGER_IN: U11.113, U15.6
- new net VDD1: C82.1, IC2.3, IC2.4, J14.3
- net 3.3V: now also C93.1, U15.8; no longer C83.1, C84.1, IC2.14, IC2.16, J15.3
- net DVDD: now also R66.2
- net GND: now also C92.2, C93.2, U15.5, U15.7
- net GND-ISO: now also C94.2, C95.2, J19.1, U15.4, U2.GND; no longer U2.1
- net N$1: now also C96.1, L6.2; no longer U2.4
- net N$2: now also C96.2, U2.0V; no longer U2.3
- net N$28: now also F1.2, L5.1; no longer R24.1, S2.3, U14.3
- net PWD: now also U11.112; no longer U11.114
- net RST: now also U11.111; no longer U11.113
- net RST_DSP: now also J18.2
- net SPI_DRDY: now also R66.1
- net VBAT: now also C83.1, C84.1, IC2.12, IC2.14, IC2.16, J15.3
- net VCC-ISO: now also F1.1; no longer U2.2
- net VCCIO: now also C94.1, U15.1, U15.3; no longer C82.1, IC2.3, IC2.4, J14.3
Routing:
- net GND-ISO: track 115.7 -> 228.8 mm, vias 1 -> 3
- net MR: track 0.00 -> 66.0 mm, vias 0 -> 2
- net VBAT: track 145.5 -> 201.7 mm, vias 3 -> 5
- net GND: track 787.9 -> 837.6 mm, vias 73 -> 82
- net N$28: track 52.0 -> 2.49 mm, vias 1 -> 0
- net ISO_IN: track 0.00 -> 46.5 mm, vias 0 -> 1
- net VCCIO: track 39.3 -> 73.4 mm
- net TRIGGER_IN: track 0.00 -> 33.0 mm
- net VCC-ISO: track 84.0 -> 115.9 mm, vias 3 -> 4
- net 3.3V: track 436.0 -> 421.8 mm
- net VDD1: track 0.00 -> 13.8 mm
- net N$2: track 9.18 -> 19.4 mm
- net RST_DSP: track 25.8 -> 34.6 mm
- net N$52: track 0.00 -> 8.09 mm
- net N$58: track 0.00 -> 6.36 mm
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- added copper zone on layer 1, net AGND
- added copper zone on layer 1, net DGND
- added copper zone on layer 16, net DGND
Other:
- board text added: "3V3"
- board text added: "GND"
- board text added: "GND-ISO"
- board text added: "GNDI"
- board text added: "ISO"
- board text added: "Jingjie Li - XJTU BME- 22 MAY 2019"
- board text added: "MR"
- board text added: "PWR"
- board text added: "RX"
- board text added: "SPD"
- board text added: "SPU"
- board text added: "TRIGGER"
- board text added: "TX"
- board text added: "V 2.1"
- board text added: "VD"
- board text removed: "Jingjie Li - XJTU BME- 11 MAY 2019"
