File: PCB/FullPCB/EEGFull.sch (EAGLE design)
At the start: 210 parts, among them IC1 ADS1299-X, IC2 ADUM4160BRWZ, J11 MICRO-SD_CARD_SOCKET, J12 455-1750-1-ND, J13 455-1750-1-ND, J14 455-1750-1-ND, J15 455-1750-1-ND, J2 USB_B_PTH, J8 JTAG, U1 LP2985-33DBVT, U10 HT7318, U11 TMS320F28335PGFA, U12 HT7333, U13 2.93V, U14 MAX811-812, U2 B0505S-1WB0505S-1W, U3 TPS60403DBVT, U4 TPS73225DBVR, U5 TPS73225DBVR, U6 TPD4E1B06DCKR, U7 TPD4E1B06DCKR, U8 TPD4E1B06DCKR, U9 HT7333, Y1 30MHz, Y2 12MHz

Commit message: update Full PCB
Parts:
- added C92, C93, C94: 0.1uF, SparkFun-Capacitors:0.1UF-0402-16V-10%
- added C95, C96: 4.7uF, SparkFun-Capacitors:4.7UF0603
- added F1: 6V/2A, SparkFun-Fuses:PPTC_HALF-AMP
- added J18: (no value), SparkFun-Connectors:CONN_02
- added J19: (no value), SparkFun-Connectors:CONN_023.5MM
- added L5, L6: 3.3µH/±20%/450mA, SparkFun-Coils:INDUCTOR-0805-3.3UH
- added R66: 10k, SparkFun-Resistors:10KOHM-0402-1/10W-1%
- added U15: ISO721D, Texas Instruments_By_element14_Batch_1:ISO721D
- U2: value B0505S-1WB0505S-1W -> B0505S-2W-SIP; device jingjieparts:B0505S-1WB0505S-1W -> jingjieparts:B0505S-2W-SIP
Connections:
- removed net PIN: IC2.PIN
- new net ISO_IN: J19.2, U15.IN
- new net MR: C92.1, J18.1, R24.1, S2.2, U14./MR
- new net N$52: C95.1, L5.2, U2.+VI
- new net N$58: L6.1, U2.+VO
- new net TRIGGER_IN: U11B.GPIO62/SCIRXDC/XD17, U15.OUT
- new net VDD1: C82.1, IC2.PDEN, IC2.VDD1, J14.3
- net 3.3V: now also C93.1, U15.VCC2; no longer C83.1, C84.1, IC2.VBUS2, IC2.VDD2, J15.3
- net DVDD: now also R66.2
- net GND: now also C92.2, C93.2, U15.GND2, U15.GND2_2
- net GND-ISO: now also C94.2, C95.2, J19.1, U15.GND1
- net N$1: now also C96.1, L6.2; no longer U2.+VO
- net N$2: now also C96.2
- net N$28: now also F1.2, L5.1; no longer R24.1, S2.2, U14./MR
- net PWD: now also U11B.GPIO61/MFSRB/XD18; no longer U11B.GPIO63/SCITXDC/XD16
- net RST: now also U11B.GPIO60/MCLKRB/XD19; no longer U11B.GPIO62/SCIRXDC/XD17
- net RST_DSP: now also J18.2
- net SPI_DRDY: now also R66.1
- net VBAT: now also C83.1, C84.1, IC2.PIN, IC2.VBUS2, IC2.VDD2, J15.3
- net VCC-ISO: now also F1.1; no longer U2.+VI
- net VCCIO: now also C94.1, U15.VCC1, U15.VCC1_2; no longer C82.1, IC2.PDEN, IC2.VDD1, J14.3
Other:
- moved on the sheet: C82, C83, C84, J3, J4, U2
